File: RAM.sch (KiCad schematic (older format))
At the start: 46 parts, among them J2 JTAG_01x06, U2 XC7K160T-FFG676, U3 MT41K512M16HA-125 :A, U4 MT41K512M16HA-125 :A, U5 TPS51200DRC, U6 KSZ9031RNXCA, U7 TUSB1310ZAY, U8 TC358867XBG, U9 SiI9022A

Commit message: some work on 6 power supplies, SPI flash
Parts:
- added C10: 0.1uF, Capacitor_SMD:C_0402_1005Metric, symbol Device:C_Small
- added C11, C12, C13, C14, C15, C16: 120p, Capacitor_SMD:C_0402_1005Metric, symbol Device:C_Small
- added L1, L2, L3, L4, L5, L6: IHLP1212AEERR47M11, Inductor_SMD:L_Vishay_IHLP-1212, symbol Device:L_Small
- added R27: 2k2, Resistor_SMD:R_0402_1005Metric, symbol Device:R_Small
- added R28, R29: 0, Resistor_SMD:R_0402_1005Metric, symbol Device:R_Small
- added R30, R31: 4k7, Resistor_SMD:R_0402_1005Metric, symbol Device:R_Small
- added R32, R35, R38, R41, R44, R47: R_Small, Resistor_SMD:R_0402_1005Metric, symbol Device:R_Small
- added R33: 453k, Resistor_SMD:R_0402_1005Metric, symbol Device:R_Small
- added R34, R37, R40, R43, R46, R49: 100k_1%, Resistor_SMD:R_0402_1005Metric, symbol Device:R_Small
- added R36: 66.5k, Resistor_SMD:R_0402_1005Metric, symbol Device:R_Small
- added R39: 200k, Resistor_SMD:R_0402_1005Metric, symbol Device:R_Small
- added R42: 150k, Resistor_SMD:R_0402_1005Metric, symbol Device:R_Small
- added R45: 83.5k, Resistor_SMD:R_0402_1005Metric, symbol Device:R_Small
- added R48: 100k, Resistor_SMD:R_0402_1005Metric, symbol Device:R_Small
- added TP1, TP2, TP3, TP4, TP5, TP6: TestPoint, symbol Connector:TestPoint
- added U10: W25Q128JVS, Package_SO:SOIC-8_5.23x5.23mm_P1.27mm, symbol Memory_Flash:W25Q128JVS
- added U11, U12, U13, U14, U15, U16: TPS62823DLC, Package_DFN_QFN:Texas_VSON-HR-8_1.5x2mm_P0.5mm, symbol Regulator_Switching:TPS62823DLC
- C1, C2, C3, C4, C5, C6, C7, C8, C9: footprint (none) -> Capacitor_SMD:C_0402_1005Metric
- D1, D2: footprint (none) -> LED_SMD:LED_0603_1608Metric
- U3, U4: symbol OrangeCrab-cache:gkl_mem_MT41K64M16TW-107_J-TR -> reform-kintex-rescue:gkl_mem_MT41K64M16TW-107_J-TR-OrangeCrab-cache
- U7: symbol TUSB1310ZAY:TUSB1310ZAY -> reform-kintex-rescue:TUSB1310ZAY-TUSB1310ZAY
- U8: symbol TC358867XBG:TC358867XBG -> reform-kintex-rescue:TC358867XBG-TC358867XBG
- U9: symbol zz9000:SiI9022A -> reform-kintex-rescue:SiI9022A-zz9000
Connections:
- net labels added: +5V, CCLK, FCS_B, QSPI_DQ0, QSPI_DQ1, QSPI_DQ2, QSPI_DQ3, SOC_RESETn
- wire segments 369 -> 522
- no-connect marks 1 -> 7
Other:
- note added: "Formula: R1 = R2 x (Vout/0.6 - 1)"
- note added: "S25FL128SAGNFI000"
- note added: "TODO: 10uF"
- note added: "TODO: 2x 10uF"
- note added: "TODO: 4.7uF"
- note added: "TODO: PUDC? \nEMCCLK?\nFCS_B?"
- note added: "TODO: according\n to ddr4 test board"
- note added: "TODO: mode straps"
- note added: "TODO: pullups?"
- note added: "antmicro use ASFLMB-100.000MHZ-XY-T"
- note added: "cost:\n~60$ fpga\n30$ memory\n5$ DP TX\n10$ USB3 PHY\n3$ HDMI TX\n15$ power"
- note removed: "TODO: QSPI flash"
- note removed: "TODO: Reset Button on PROGRAM_B"
- note removed: "cost:\n~60$ fpga\n30$ memory\n5$ DP TX\n10$ USB3 PHY\n3$ HDMI TX\n"
- moved on the sheet: D1, D2, R22, R23, R24, R25

Commit message: switch to TC358778XBG, some more connections here and there
Parts:
- removed U8: TC358867XBG, footprints:BGA80C65P10X10_700X700X100, symbol reform-kintex-rescue:TC358867XBG-TC358867XBG
- added C? (x5): 10uF, symbol Device:C_Small
- added C?: 0.1uF, symbol Device:C_Small
- added C?: 1nF, symbol Device:C_Small
- added C? (x4): 10nF, symbol Device:C_Small
- added C?: 0.1uF, Capacitor_SMD:C_0402_1005Metric, symbol Device:C_Small
- added C? (x2): 22pF, symbol Device:C_Small
- added R? (x4): 10k, symbol Device:R_Small
- added R?: 12.1k, symbol Device:R_Small
- added R?: 1.8M, symbol Device:R_Small
- added U?: TC358778XBG, BGA80C65P10X10_700X700X100, symbol reform2-som:TC358778XBG
- added Y?: ABM8G-25.000MHZ-18-D2Y-T, symbol Device:Crystal_GND24_Small
- U3, U4: value MT41K512M16HA-125 :A -> IS43TR16512B-125KBLI
Connections:
- net labels added: DISP1_CLK, DISP1_IRQ, DSI_CLK_N, DSI_CLK_P, DSI_D0_N, DSI_D0_P, DSI_D1_N, DSI_D1_P, DSI_D2_N, DSI_D2_P, DSI_D3_N, DSI_D3_P, DSI_RST_N, ETH0_LED_LINK1, ETH0_LED_RX, ETH_INT_N, ETH_MDC, ETH_MDIO, ETH_REF_CLK, ETH_RX_CLK, ETH_RX_DV, I2C1_SCL, I2C1_SDA, VTTREF
- net labels removed: DPAUX+, DPAUX-, DPLN0+, DPLN0-, DPLP1+, DPLP1-
- wire segments 522 -> 887
- no-connect marks 7 -> 15
Other:
- note added: "Config Flash"
- note added: "DDR3 RAM"
- note added: "ETHERNET"
- note added: "HDMI"
- note added: "IS43TR16512B-125KBLI"
- note added: "MIPI-DSI"
- note added: "TODO: A5 was here"
- note added: "TODO: Pullups and Pulldowns"
- note added: "TODO: REFCLK"
- note added: "TODO: floorplan"
- note added: "TODO: wrong balls"
- note added: "USB"
- note added: "cost:\n~60$ fpga\n30$ memory\n7$ DSI TX\n10$ USB3 PHY\n3$ HDMI TX\n15$ power"
- note added: "current specs:\n- Kintex-7 XC7K160T (can also be swapped with some others)\n- 2GB DDR3\n- 2x PCIe (to M.2 and mPCIe on motherboad)\n- USB3,2\n- HDMI (1080p for now)\n- MIPI-DSI (1080p)\n- Ethernet (1Gbe)\n- SPI flash\n- Interfaces to SD card, SAI, UART, JTAG on motherboard"
- note removed: "25mhz crystal?"
- note removed: "RX pullups?"
- note removed: "TODO: 1V5?"
- note removed: "TODO: ETH?"
- note removed: "TODO: VREF in GENESYS"
- note removed: "cost:\n~60$ fpga\n30$ memory\n5$ DP TX\n10$ USB3 PHY\n3$ HDMI TX\n15$ power"
- moved on the sheet: C1, C10, D1, D2, J2, R1, R10, R11, R12, R13, R14, R15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

Commit message: some more TUSB signals connected
Parts:
- added C? (x2): 22pF, symbol Device:C_Small
- added R?: 10k 1%, symbol Device:R_Small
- added R?: 90.9k 1%, symbol Device:R_Small
- added R?: 1.8M, symbol Device:R_Small
- added TP?: TestPoint, symbol Connector:TestPoint
- added TP?: TUSBJ_TCK, symbol Connector:TestPoint
- added TP?: TUSBJ_TMS, symbol Connector:TestPoint
- added TP?: TUSBJ_TDI, symbol Connector:TestPoint
- added TP?: TUSBJ_TRSTN, symbol Connector:TestPoint
- added TP?: TUSBJ_TDO, symbol Connector:TestPoint
- added Y?: ABM8G-20.000MHZ-18-D2Y-T, symbol Device:Crystal_GND24_Small
- U?: symbol reform2-som:TC358778XBG -> reform-kintex-rescue:TC358778XBG-reform2-som
Connections:
- net labels added: TUSB_ENAB, TUSB_PHYRESETN, TUSB_RESETN, TUSB_RX_D0, TUSB_RX_D1, TUSB_RX_D10, TUSB_RX_D11, TUSB_RX_D12, TUSB_RX_D13, TUSB_RX_D14, TUSB_RX_D15, TUSB_RX_D2, TUSB_RX_D3, TUSB_RX_D4, TUSB_RX_D5, TUSB_RX_D6, TUSB_RX_D7, TUSB_RX_D8, TUSB_RX_D9, TUSB_TX_D0, TUSB_TX_D1, TUSB_TX_D10, TUSB_TX_D11, TUSB_TX_D12, TUSB_TX_D13, TUSB_TX_D14, TUSB_TX_D2, TUSB_TX_D3, TUSB_TX_D4, TUSB_TX_D5, TUSB_TX_D6, TUSB_TX_D7, TUSB_TX_D8, TUSB_TX_D9, TUSB_ULPI_D0, TUSB_ULPI_D1, TUSB_ULPI_D2, TUSB_ULPI_D3, TUSB_ULPI_D4, TUSB_ULPI_D5, TUSB_ULPI_D6, TUSB_ULPI_D7, TUSB_ULPI_DIR
- wire segments 887 -> 1030
Other:
- note added: "TODO: up to 40MHz"
- moved on the sheet: U7A, U7C

Commit message: more TUSB noodling
Parts:
- added C? (x2): 4.7nF, symbol Device:C_Small
- added R? (x2): 10k, symbol Device:R_Small
- added R?: 0, symbol Device:R_Small
- added R?: 10k 1%, symbol Device:R_Small
Connections:
- net +1V8: now also R?.1
- net GND: now also C?.2, C?.2, R?.1
- net TUSB_RX_STAT0: now reaches U7.C5 (RX_STATUS0)
- net TUSB_RX_STAT1: now reaches U7.C6 (RX_STATUS1)
- net TUSB_RX_STAT2: now reaches U7.C7 (RX_STATUS2)
- net TUSB_RX_POLARITY: now reaches U7.C8 (RX_POLARITY)
- net TUSB_PHY_STATUS: now reaches U7.E3 (PHY_STATUS)
- net TUSB_RX_ELECIDLE: now reaches U7.F3 (RX_ELECIDLE)
- net TUSB_TX_DATAK1: now reaches U7.G1 (TX_DATAK1)
- net TUSB_PDOWN1: now reaches U7.G3 (POWER_DOWN1)
- net TUSB_PDOWN0: now reaches U7.H3 (POWER_DOWN0)
- net TUSB_TX_DATAK0: now reaches U7.J1 (TX_DATAK0)
- net TUSB_TXCLK: now reaches U7.K1 (TX_CLK)
- net TUSB_TX_DEEMPH1: now reaches U7.K11 (TX_DEEMPH1)
- net TUSB_TX_ELECIDLE: now reaches U7.K3 (TX_ELECIDLE)
- net TUSB_TX_DEEMPH0: now reaches U7.L11 (TX_DEEMPH0)
- net TUSB_TX_MARGIN1: now reaches U7.M10 (TX_MARGIN1)
- net TUSB_TX_MARGIN2: now reaches U7.M11 (TX_MARGIN2)
- net TUSB_ONEZERO: now reaches U7.M4 (TX_ONESZEROS)
- net TUSB_TX_SWING: now reaches U7.M5 (TX_SWING)
- net TUSB_TX_MARGIN0: now reaches U7.M9 (TX_MARGIN0)
- net at U7.A14 (CEXTSS): now also C?.1
- net at U7.D10 (CLKOUT): now also R?.1
- net at U7.H12 (PHY_MODE1): now also R?.2
- net at U7.J12 (PHY_MODE0): now also R?.2
- net at U7.L13 (R1EXTRTN): now also R?.2
- net at U7.L14 (R1EXT): now also R?.1
- net at U7.M14 (CEXT): now also C?.1
- new net TUSB_CLKOUT: R?.2
Other:
- moved on the sheet: R?

Commit message: finish first draft of TUSB connectivity
Parts:
- added C? (x2): 0.1uF, symbol Device:C_Small
- added R? (x12): DNP, symbol Device:R_Small
Connections:
- net labels added: TUSB_PCLK, TUSB_PWRPRESENT, TUSB_RX_K0, TUSB_RX_K1, TUSB_RX_VALID, TUSB_TX_D15, TUSB_TX_DETRX_LPBK, TUSB_ULPI_CLK, TUSB_ULPI_NXT, TUSB_ULPI_STP, TUSB_VSSOSC
- net labels removed: TUSB_ONEZERO, TUSB_RX_POLARITY, TUSB_TX_DEEMPH0, TUSB_TX_DEEMPH1, TUSB_TX_MARGIN0, TUSB_TX_MARGIN1, TUSB_TX_MARGIN2, TUSB_TX_SWING
- wire segments 1070 -> 1159
- no-connect marks 15 -> 20
Other:
- note added: "TODO: PCIe clocking"
- note added: "TUSB is ULPI master"
- moved on the sheet: R?, U2A, U2B, U2C

Commit message: more DDR3 routing
Parts:
- added J3: Conn_01x03_Male, symbol Connector:Conn_01x03_Male
- added R75: 4.7k, Resistor_SMD:R_0402_1005Metric, symbol Device:R_Small
- added R76: 330, Resistor_SMD:R_0402_1005Metric, symbol Device:R_Small
- added R77: 100, Resistor_SMD:R_0402_1005Metric, symbol Device:R_Small
- added R78, R82, R83: DNP, Resistor_SMD:R_0402_1005Metric, symbol Device:R_Small
- added R79, R80, R81: 0, Resistor_SMD:R_0402_1005Metric, symbol Device:R_Small
- C17, C18, C19, C20, C21, C22, C23, C24, C25, C26, C27, C29, C30, C31, C32, C33, C34, C35, C36: renamed from C?; footprint (none) -> Capacitor_SMD:C_0402_1005Metric
- R23: value 4.7k -> ???
- R50, R51, R52, R53, R54, R55, R56, R57, R58, R59, R60, R61, R62, R63, R64, R65, R66, R67, R68, R69, R70, R71, R72, R73, R74: renamed from R?; footprint (none) -> Resistor_SMD:R_0402_1005Metric
- U8: renamed from U?; footprint BGA80C65P10X10_700X700X100 -> footprints:BGA80C65P10X10_700X700X100
- U9: footprint footprints:QFN50P700X700X100-49N -> Package_DFN_QFN:QFN-72-1EP_10x10mm_P0.5mm_EP6x6mm
- gave numbers to parts that had none: 9
Connections:
- net labels added: MODE0, MODE1, MODE2, PUDC_B, USB1TXN, USB1TXP
- wire segments 1159 -> 1170
- no-connect marks 20 -> 22
Other:
- note removed: "TODO: mode straps"
- note removed: "TODO: pullups?"
- moved on the sheet: D1, D2, R22, R23, R24, R25
