File: RAM.sch (KiCad schematic (older format))
At the start: 344 parts, among them J2 JTAG_01x06, J3 Conn_01x03_Male, U10 W25Q128JVS, U11 TPS62823DLC, U12 TPS62823DLC, U13 TPS62823DLC, U14 TPS62823DLC, U15 TPS62823DLC, U16 TPS62823DLC, U17 Si52112-B6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

Commit message: silkscreen cleanup, 3d models, some footprint fixes
Parts:
- U17: value Si52112-B6 -> Si52112-B5-GM2; footprint Package_DFN_QFN:TDFN-8-1EP_3x2mm_P0.5mm_EP1.3x1.4mm -> footprints:Silicon_Labs-Si52112-B5-GM2-Level_B; symbol reform2-som:Si52112-B6 -> reform2-som:Si52112-B5
- X1: footprint Oscillator:Oscillator_SMD_Abracon_ASE-4Pin_3.2x2.5mm -> footprints:OSCDFN500X320X90-4N
Connections:
- net +3V3: now also U17.10 (VDD)
- net GND: now also U17.5 (VSS)
- net PCIE1_CLK_HOST_N: now also U17.7 (~DIFF1); no longer U17.6 (~DIFF1)
- net PCIE1_CLK_HOST_P: now also U17.6 (DIFF1); no longer U17.5 (DIFF1)
- net PCIE1_CLK_N: now also U17.9 (~DIFF2); no longer U17.8 (~DIFF2)
- net PCIE1_CLK_P: now also U17.8 (DIFF2); no longer U17.7 (DIFF2)
- net EDP_RESETn: now reaches U2.C14 (IO_L19P_T3_16)
- net USB_RESETn: now reaches U2.D13 (IO_L17N_T2_16)
Other:
- note added: "DNP?"
- note removed: "TODO: REFCLK"
- moved on the sheet: C191, C88, Y3
Changed lines of the file:
@@
 Text GLabel 16800 3500 2    50   Output ~ 0
 DISP2_DE
-Text GLabel 21500 12700 2    50   Output ~ 0
-PCIE1_CLK_N
 Text GLabel 21500 12850 2    50   Output ~ 0
+PCIE1_CLK_N
+Text GLabel 21500 13000 2    50   Output ~ 0
 PCIE1_CLK_P
 Text GLabel 19000 11850 2    50   Input ~ 0
@@
 Wire Wire Line
 	32350 11300 32200 11300
-Text Notes 29500 9000 0    50   ~ 0
-TODO: REFCLK
 Text Notes 31050 8450 0    50   ~ 0
 MIPI-DSI
@@
 	18150 11750 17400 11750
 $Comp
-L reform2-som:Si52112-B6 U17
+L reform2-som:Si52112-B5 U17
 U 1 1 70F5A39F
 P 20850 12900
 F 0 "U17" H 20850 13365 50  0000 C CNN
-F 1 "Si52112-B6" H 20850 13274 50  0000 C CNN
-F 2 "Package_DFN_QFN:TDFN-8-1EP_3x2mm_P0.5mm_EP1.3x1.4mm" H 20850 12450 50  0001 C CNN
+F 1 "Si52112-B5-GM2" H 20850 13274 50  0000 C CNN
+F 2 "footprints:Silicon_Labs-Si52112-B5-GM2-Level_B" H 20850 12450 50  0001 C CNN
 F 3 "" H 20850 12450 50  0001 C CNN
 	1    20850 12900
@@
 L power:+3V3 #PWR073
 U 1 1 70F6B46D
-P 21350 13600
-F 0 "#PWR073" H 21350 13450 50  0001 C CNN
-F 1 "+3V3" H 21365 13773 50  0000 C CNN
-F 2 "" H 21350 13600 50  0001 C CNN
-F 3 "" H 21350 13600 50  0001 C CNN
-	1    21350 13600
+P 21350 13700
+F 0 "#PWR073" H 21350 13550 50  0001 C CNN
+F 1 "+3V3" H 21365 13873 50  0000 C CNN
+F 2 "" H 21350 13700 50  0001 C CNN
+F 3 "" H 21350 13700 50  0001 C CNN
+	1    21350 13700
 	1    0    0    -1
 $EndComp
 Wire Wire Line
-	21350 13600 21350 13750
+	21350 13700 21350 13750
 Wire Wire Line
 	21350 13750 21700 13750
@@
 Wire Wire Line
 	18900 11650 19000 11650
-Text GLabel 21500 13150 2    50   Output ~ 0
+Text GLabel 21500 13300 2    50   Output ~ 0
 PCIE1_CLK_HOST_P
-Text GLabel 21500 13000 2    50   Output ~ 0
+Text GLabel 21500 13150 2    50   Output ~ 0
 PCIE1_CLK_HOST_N
 Wire Wire Line
@@
 $EndComp
 Wire Wire Line
-	19850 13900 19700 13900
-Connection ~ 19850 13900
+	19850 14150 19700 14150
+Connection ~ 19850 14150
 Wire Wire Line
-	19850 13350 19850 13900
+	19850 13350 19850 14150
 Wire Wire Line
 	19700 13350 19850 13350
 Wire Wire Line
-	19700 13400 19700 13350
-Connection ~ 19300 13500
-Connection ~ 20100 13500
+	19700 13650 19700 13350
+Connection ~ 19300 13750
+Connection ~ 20100 13750
 Wire Wire Line
-	20100 13500 19800 13500
+	20100 13750 19800 13750
 Wire Wire Line
-	20100 13600 20100 13500
+	20100 13850 20100 13750
 Wire Wire Line
-	20100 13900 19850 13900
+	20100 14150 19850 14150
 Wire Wire Line
-	20100 13800 20100 13900
+	20100 14050 20100 14150
 $Comp
 L Device:C_Small C191
 U 1 1 6492DDEE
-P 20100 13700
-F 0 "C191" H 20192 13746 50  0000 L CNN
-F 1 "22pF" H 20192 13655 50  0000 L CNN
-F 2 "Capacitor_SMD:C_0402_1005Metric" H 20100 13700 50  0001 C CNN
-F 3 "~" H 20100 13700 50  0001 C CNN
-	1    20100 13700
+P 20100 13950
+F 0 "C191" H 20192 13996 50  0000 L CNN
+F 1 "22pF" H 20192 13905 50  0000 L CNN
+F 2 "Capacitor_SMD:C_0402_1005Metric" H 20100 13950 50  0001 C CNN
+F 3 "~" H 20100 13950 50  0001 C CNN
+	1    20100 13950
 	1    0    0    -1
 $EndComp
 Wire Wire Line
-	19700 13900 19700 13600
-Connection ~ 19700 13900
+	19700 14150 19700 13850
+Connection ~ 19700 14150
 Wire Wire Line
-	19300 13900 19700 13900
+	19300 14150 19700 14150
 Wire Wire Line
-	19300 13800 19300 13900
+	19300 14050 19300 14150
 Wire Wire Line
-	19700 13950 19700 13900
+	19700 14200 19700 14150
 $Comp
 L power:GND #PWR0182
 U 1 1 6492DDFD
-P 19700 13950
-F 0 "#PWR0182" H 19700 13700 50  0001 C CNN
-F 1 "GND" H 19705 13777 50  0000 C CNN
-F 2 "" H 19700 13950 50  0001 C CNN
-F 3 "" H 19700 13950 50  0001 C CNN
-	1    19700 13950
+P 19700 14200
+F 0 "#PWR0182" H 19700 13950 50  0001 C CNN
+F 1 "GND" H 19705 14027 50  0000 C CNN
+F 2 "" H 19700 14200 50  0001 C CNN
+F 3 "" H 19700 14200 50  0001 C CNN
+	1    19700 14200
 	1    0    0    -1
 $EndComp
 Wire Wire Line
-	19300 13500 19300 13600
+	19300 13750 19300 13850
 Wire Wire Line
-	19600 13500 19300 13500
+	19600 13750 19300 13750
 $Comp
 L Device:C_Small C88
 U 1 1 6492DE09
-P 19300 13700
-F 0 "C88" H 19392 13746 50  0000 L CNN
-F 1 "22pF" H 19392 13655 50  0000 L CNN
-F 2 "Capacitor_SMD:C_0402_1005Metric" H 19300 13700 50  0001 C CNN
-F 3 "~" H 19300 13700 50  0001 C CNN
-	1    19300 13700
+P 19300 13950
+F 0 "C88" H 19392 13996 50  0000 L CNN
+F 1 "22pF" H 19392 13905 50  0000 L CNN
+F 2 "Capacitor_SMD:C_0402_1005Metric" H 19300 13950 50  0001 C CNN
+F 3 "~" H 19300 13950 50  0001 C CNN
+	1    19300 13950
 	1    0    0    -1
 $EndComp
@@
 L Device:Crystal_GND24_Small Y3
 U 1 1 6492DE13
-P 19700 13500
-F 0 "Y3" H 19844 13546 50  0000 L CNN
-F 1 "ABM8G-25.000MHZ-18-D2Y-T" H 19844 13455 50  0000 L CNN
-F 2 "Crystal:Crystal_SMD_3225-4Pin_3.2x2.5mm" H 19700 13500 50  0001 C CNN
-F 3 "~" H 19700 13500 50  0001 C CNN
-	1    19700 13500
+P 19700 13750
+F 0 "Y3" H 19844 13796 50  0000 L CNN
+F 1 "ABM8G-25.000MHZ-18-D2Y-T" H 19844 13705 50  0000 L CNN
+F 2 "Crystal:Crystal_SMD_3225-4Pin_3.2x2.5mm" H 19700 13750 50  0001 C CNN
+F 3 "~" H 19700 13750 50  0001 C CNN
+	1    19700 13750
 	1    0    0    -1
 $EndComp
@@
 L power:GND #PWR0185
 U 1 1 65F4DAE9
-P 20300 13200
-F 0 "#PWR0185" H 20300 12950 50  0001 C CNN
-F 1 "GND" H 20305 13027 50  0000 C CNN
-F 2 "" H 20300 13200 50  0001 C CNN
-F 3 "" H 20300 13200 50  0001 C CNN
-	1    20300 13200
+P 20300 13400
+F 0 "#PWR0185" H 20300 13150 50  0001 C CNN
+F 1 "GND" H 20305 13227 50  0000 C CNN
+F 2 "" H 20300 13400 50  0001 C CNN
+F 3 "" H 20300 13400 50  0001 C CNN
+	1    20300 13400
 	1    0    0    -1
 $EndComp
 Wire Wire Line
-	20300 13200 20300 13150
-Wire Wire Line
 	20300 13150 20350 13150
 $Comp
@@
 	20100 13000 20350 13000
 Wire Wire Line
-	20100 13000 20100 13500
+	20100 13000 20100 13750
 Wire Wire Line
 	19300 12850 20350 12850
 Wire Wire Line
-	19300 12850 19300 13500
+	19300 12850 19300 13750
 $Comp
 L Oscillator:ASE-xxxMHz X1
@@
 F 0 "X1" H 34050 6350 50  0000 L CNN
 F 1 "ASFLMB-100.000MHZ-XY-T" H 34050 6000 50  0000 L CNN
-F 2 "Oscillator:Oscillator_SMD_Abracon_ASE-4Pin_3.2x2.5mm" H 34500 5800 50  0001 C CNN
+F 2 "footprints:OSCDFN500X320X90-4N" H 34500 5800 50  0001 C CNN
 F 3 "http://www.abracon.com/Oscillators/ASV.pdf" H 33700 6150 50  0001 C CNN
 	1    33800 6150
@@
 Text GLabel 11300 2300 2    50   Output ~ 0
 BACKLIGHT_EN
+Text Notes 24850 14350 0    50   ~ 0
+DNP?
+Text Notes 25550 14350 0    50   ~ 0
+DNP?
+Text GLabel 12800 5500 0    50   Output ~ 0
+USB_RESETn
+Text GLabel 12800 5800 0    50   Output ~ 0
+EDP_RESETn
+Wire Wire Line
+	21350 13300 21500 13300
+$Comp
+L power:+3V3 #PWR0195
+U 1 1 8C067089
+P 21500 12700
+F 0 "#PWR0195" H 21500 12550 50  0001 C CNN
+F 1 "+3V3" H 21515 12873 50  0000 C CNN
+F 2 "" H 21500 12700 50  0001 C CNN
+F 3 "" H 21500 12700 50  0001 C CNN
+	1    21500 12700
+	1    0    0    -1
+$EndComp
+Wire Wire Line
+	20350 13300 20300 13300
+Wire Wire Line
+	20300 13150 20300 13300
+Wire Wire Line
+	20300 13300 20300 13400
+Connection ~ 20300 13300
 $EndSCHEMATC

Commit message: DRC, polishing, bugfixes, badge
Parts:
- added GFX2: MountingHole, footprints:mnt-rkx7-badge-d01, symbol Mechanical:MountingHole
- added R105, R106, R107, R108: 4.7k, Resistor_SMD:R_0402_1005Metric, symbol Device:R_Small
- added R109: 4k7, Resistor_SMD:R_0402_1005Metric, symbol Device:R_Small
- C82, C89, C93, C94, C97, C98: footprint Capacitor_SMD:C_0402_1005Metric -> Capacitor_SMD:C_0603_1608Metric
- GFX1: footprint footprints:mnt-kx7000 -> footprints:mnt-rkx7
- R23: value ??? -> 4.7k
- U6: value KSZ9031RNXCA -> KSZ9031RNX
Connections:
- net +1V2: now also U9.66 (AVCC12)
- net +1V8: now also U9.69 (IO_SEL), R109.1
- net +3V3: now also R105.1, R106.1, R107.1
- net DSI_REFCLK: now also U2.AD18 (IO_L13N_T2_MRCC_32)
- net ETH_RX_D0: now also R108.1
- net ETH_RX_D1: now also R105.2
- net ETH_RX_D2: now also R106.2
- net ETH_RX_D3: now also R107.2
- net GND: now also U2.M11 (GNDADC_0), R108.2; no longer U9.69 (IO_SEL)
- net USB1TXN: now also C33.2, U7.J14 (SSTXM); no longer C31.2, U7.H14 (SSTXP)
- net USB1TXP: now also C31.2, U7.H14 (SSTXP); no longer C33.2, U7.J14 (SSTXM)
- net USB1_RX_N: now also U7.F14 (SSRXM); no longer U7.E14 (SSRXP)
- net USB1_RX_P: now also U7.E14 (SSRXP); no longer U7.F14 (SSRXM)
- net USB1_TX_N: now also C33.1; no longer C31.1
- net USB1_TX_P: now also C31.1; no longer C33.1
- net at U9.72 (CI2CA): now also R109.2
- net DISP1_IRQ: no longer names the net of U9.52 (INT)
- net VAA: no longer names the net of TP7.1, U2.P12 (VREFP_0)
- no-connect marks 77 -> 193
Other:
- note added: "Config Bank Voltage Select"
- note added: "Config: 1110 (RGMII)"
- note removed: "0.75V Vtt"
- note removed: "200MHz sysclock: DSC1103CE2-200.0?"
- note removed: "TODO: 0603"
- note removed: "TODO: PUDC? \nEMCCLK?\nFCS_B?"
- note removed: "TODO: Pullups and Pulldowns"
- note removed: "TODO: bank 14 config pins"
- note removed: "TODO: double check CI2CA"
- note removed: "TODO: double check,\nreally 3v3?"
- note removed: "TODO: double check.\nkinda weird locations."
- note removed: "TODO: series Rs?"
- note removed: "TODO: wrong balls"
- note removed: "actually KSZ9131RNX"
- moved on the sheet: TP7

Commit message: add readme, schematics pdf, image
Other:
- note removed: "S25FL128SAGNFI000"
- note removed: "cost:\n~60$ fpga\n30$ memory\n7$ DSI TX\n10$ USB3 PHY\n3$ HDMI TX\n15$ power"
- note removed: "current specs:\n- Kintex-7 XC7K160T (can also be swapped with some others)\n- 2GB DDR3\n- 2x PCIe (to M.2 and mPCIe on motherboad)\n- USB3,2\n- HDMI (1080p for now)\n- MIPI-DSI (1080p)\n- Ethernet (1Gbe)\n- SPI flash\n- Interfaces to SD card, SAI, UART, JTAG on motherboard"
- moved on the sheet: C1, C10, C100, C101, C102, C103, C104, C105, C106, C107, C108, C109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

Commit message: WIP adjust ddr trace widths; prepare some TODOs for errors found with vivado
Parts:
- U17: symbol reform2-som:Si52112-B5 -> reform-kintex-rescue:Si52112-B5-reform2-som
Connections:
- no-connect marks 193 -> 192
Other:
- note added: "TODO: move 100 mhz clkin to this column"
- note added: "TODO: move syclk here"
- note added: "TODO: validate pin assignment in vivado"
Changed lines of the file:
@@
 Text GLabel 7000 12600 2    50   Input ~ 0
 RAM_D15
-Text GLabel 7000 11300 2    50   Input ~ 0
+Text GLabel 7000 12900 2    50   Input ~ 0
 RAM_D13
-Text GLabel 7000 11700 2    50   Input ~ 0
-RAM_D11
 Text GLabel 7000 12500 2    50   Input ~ 0
+RAM_D11
+Text GLabel 7000 11700 2    50   Input ~ 0
 RAM_D7
 Text GLabel 7000 13300 2    50   Input ~ 0
 RAM_D10
-Text GLabel 7000 11400 2    50   Input ~ 0
+Text GLabel 7000 13000 2    50   Input ~ 0
 RAM_D9
 Text GLabel 7000 12400 2    50   Input ~ 0
 RAM_D8
-Text GLabel 7000 12900 2    50   Input ~ 0
+Text GLabel 7000 11300 2    50   Input ~ 0
 RAM_D5
 Text GLabel 7000 11900 2    50   Input ~ 0
 RAM_D4
-Text GLabel 7000 13000 2    50   Input ~ 0
+Text GLabel 7000 11400 2    50   Input ~ 0
 RAM_D3
 Text GLabel 7000 11200 2    50   Input ~ 0
@@
 Text GLabel 7000 13400 2    50   Input ~ 0
 RAM_RESET#
-Text GLabel 7000 14600 2    50   Input ~ 0
-RAM_DM1
 Text GLabel 3000 13400 0    50   Input ~ 0
 RAM_CS#
@@
 	19100 13350 18350 13350
 $Comp
-L reform2-som:Si52112-B5 U17
+L reform-kintex-rescue:Si52112-B5-reform2-som U17
 U 1 1 70F5A39F
 P 21800 14500
+AR Path="/70F5A39F" Ref="U17"  Part="1"
+AR Path="/5FC501AB/70F5A39F" Ref="U17"  Part="1"
 F 0 "U17" H 21800 14965 50  0000 C CNN
 F 1 "Si52112-B5-GM2" H 21800 14874 50  0000 C CNN
@@
 Wire Wire Line
 	9650 22550 10450 22550
-NoConn ~ 7000 12300
 NoConn ~ 3000 13800
 NoConn ~ 3000 13700
@@
 	1    0    0    -1
 $EndComp
+Text Notes 750  11550 0    50   ~ 0
+TODO: move 100 mhz clkin to this column
+Text Notes 750  11400 0    50   ~ 0
+TODO: validate pin assignment in vivado
+Text GLabel 7000 12300 2    50   Input ~ 0
+RAM_DM1
+Text Notes 1850 13750 0    50   ~ 0
+TODO: move syclk here
 $EndSCHEMATC
