File: reform-kintex.kicad_sch (KiCad schematic)
At the start: 3 parts, among them U1 MNT Reform 2.0 SoM Socket

Commit message: clean up schematics
Other:
- sheet RAM renamed FPGA, RAM, Support
- note added: "MNT REFORM CPU CONNECTOR"
- moved on the sheet: H1, H2, U1
